File: Hardware/sled/sled.kicad_pcb (KiCad board)
At the start: 4 copper layers, 185.2 x 33 mm, 29 parts, among them J1 LEO2, J10 DCDC1, J11 Ezmini1, J2 LEO1, J4 Strat1, J5 Ezmini1, J7 FWGPS, J8 camera, J9 DCDC1, SW1 SW_DPST_x2, SW2 SW_DPST_x2

Commit message: work
Parts:
- added G***: LOGO, LOGO, F.Cu at (187.8, 69.1)
Other:
- copper layers 4 -> 2
- board text added: "2s batt +-"
- board text added: "cam +-"
- board text added: "easymini"
- board text added: "ez -+"
- board text added: "fw +-"
- board text added: "gps"
- board text added: "inconverter"
- board text added: "leo"
- board text added: "strat"
- board text added: "strat -+"
